File: HandiFinder.brd (EAGLE design)
At the start: 30.1 x 59.7 mm, 25 parts, among them IC2 4047D, X1 SMA-142-0701-801/806

Commit message: Change hole diameter to 2.6mm to allow 2.5mm screw. Change diode footprint to SOD 123.
Parts:
- removed ANT1GND, ANT2, ANT2GND: WIREPAD4,16O1,6, wirepad:4,16O1,6
- added ANT1GND2, ANT22, ANT2GND2: WIREPAD, wirepad2.6:2.6MMHOLE
- ANT1: value WIREPAD4,16O1,6 -> ANT12; device wirepad:4,16O1,6 -> wirepad2.6:2.6MMHOLE
- D1, D2: value 1N4148WS -> 1N4148; device Diodes:SOD-323 -> Seeed-Diode-2016:SOD-123
- turned D1 to 0 degrees
- turned D2 to 180 degrees
Connections:
- net GND: now also ANT1GND2.P$1, ANT2GND2.P$1; no longer ANT1GND.1, ANT2GND.1
- net N$10: now also D1.+, D2.+; no longer D1.A, D2.A
- net N$11: now also D1.-; no longer D1.C
- net N$14: now also ANT1.P$1; no longer ANT1.1
- net N$15: now also ANT22.P$1; no longer ANT2.1
- net N$4: now also D2.-; no longer D2.C
Routing:
- net N$10: track 25.2 -> 24.0 mm
Other:
- board text added: "Ant1"
- board text added: "Ant2"
- board text added: "GND1"
- board text added: "GND2"
- board text added: "Handi Finder PCB by F4HVO 1.1 09/2019"
- board text removed: "Handi Finder PCB by F4HVO 1.0 08/2019"
