File: HandiFinder.brd (EAGLE design)
At the start: 30.1 x 59.7 mm, 25 parts, among them IC2 4047D, X1 SMA-142-0701-801/806

Commit message: Fix switch misconnection.
Connections:
- net +5V: no longer IC2.14
- net N$16: now also IC2.14
Routing:
- net +5V: track 47.5 -> 32.3 mm
- net N$16: track 40.3 -> 49.0 mm
Other:
- board text added: "Handi Finder PCB by F4HVO 1.2 10/2019"
- board text removed: "Handi Finder PCB by F4HVO 1.1 09/2019"
Changed lines of the file:
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@@
 <text x="2.54" y="38.1" size="1.778" layer="22" rot="MR180">Handi Finder
 PCB by F4HVO
-1.1 09/2019</text>
+1.2 10/2019</text>
 <text x="1.27" y="74.93" size="1.778" layer="25">Ant1</text>
 <text x="24.13" y="74.93" size="1.778" layer="25">Ant2</text>
@@
 <element name="D1" library="Seeed-Diode-2016" package="SOD-123" value="1N4148" x="20.32" y="57.15" smashed="yes">
 <attribute name="MPN" value="MMSD4148" x="20.32" y="57.15" size="1.778" layer="27" display="off"/>
+<attribute name="NAME" x="18.415" y="58.293" size="0.889" layer="25" ratio="11"/>
 <attribute name="NAME" x="19.431" y="56.515" size="0.381" layer="33" ratio="10"/>
-<attribute name="NAME" x="18.415" y="58.293" size="0.889" layer="25" ratio="11"/>
 <attribute name="VALUE" x="18.415" y="55.118" size="0.889" layer="27" font="vector" ratio="11"/>
 </element>
 <element name="D2" library="Seeed-Diode-2016" package="SOD-123" value="1N4148" x="10.16" y="57.15" smashed="yes" rot="R180">
 <attribute name="MPN" value="MMSD4148" x="10.16" y="57.15" size="1.778" layer="27" rot="R180" display="off"/>
+<attribute name="NAME" x="12.065" y="56.007" size="0.889" layer="25" ratio="11" rot="R180"/>
 <attribute name="NAME" x="11.049" y="57.785" size="0.381" layer="33" ratio="10" rot="R180"/>
-<attribute name="NAME" x="12.065" y="56.007" size="0.889" layer="25" ratio="11" rot="R180"/>
 <attribute name="VALUE" x="12.065" y="59.182" size="0.889" layer="27" font="vector" ratio="11" rot="R180"/>
 </element>
@@
 <signal name="+5V">
 <contactref element="9V" pad="1"/>
-<contactref element="IC2" pad="14"/>
 <contactref element="S1" pad="2"/>
-<wire x1="11.2776" y1="37.30101875" x2="11.2776" y2="38.0238" width="0.6096" layer="1"/>
-<wire x1="11.2776" y1="38.0238" x2="10.795" y2="38.5064" width="0.6096" layer="1"/>
-<wire x1="24.384" y1="35.56" x2="13.01861875" y2="35.56" width="0.6096" layer="1"/>
-<wire x1="13.01861875" y1="35.56" x2="11.2776" y2="37.30101875" width="0.6096" layer="1"/>
 <wire x1="10.16" y1="25.4" x2="12.7" y2="22.86" width="0.6096" layer="1"/>
 <wire x1="22.86" y1="22.86" x2="22.86" y2="29.21" width="0.6096" layer="1"/>
@@
 <via x="20.32" y="30.48" extent="1-16" drill="0.35"/>
 <wire x1="20.32" y1="30.48" x2="20.32" y2="33.02" width="0.6096" layer="1"/>
+<contactref element="IC2" pad="14"/>
+<wire x1="15.875" y1="33.4264" x2="15.875" y2="32.3596" width="0.6096" layer="1"/>
+<wire x1="10.795" y1="38.5064" x2="11.2776" y2="38.0238" width="0.6096" layer="1"/>
+<wire x1="11.2776" y1="38.0238" x2="11.2776" y2="37.30101875" width="0.6096" layer="1"/>
+<wire x1="11.2776" y1="37.30101875" x2="11.54541875" y2="37.0332" width="0.6096" layer="1"/>
+<wire x1="11.54541875" y1="37.0332" x2="12.2682" y2="37.0332" width="0.6096" layer="1"/>
+<wire x1="12.2682" y1="37.0332" x2="15.875" y2="33.4264" width="0.6096" layer="1"/>
 </signal>
 </signals>
